File: PecanPico6.sch (EAGLE design)
At the start: 80 parts, among them IC1 TPS79718DCKT, IC2 SI4463/4, IC3 UBLOX_MAX-6, IC4 LPC1114FHN33/333, IC5 SPV1040, IC6 AS213-92LF, IC7 BMP180, Q2 AP2301

Commit message: Corrected 'UART TXD,RXD switched' error
Connections:
- net RXD: now also SJ2.2; no longer SJ1.2
- net TXD: now also SJ1.2; no longer SJ2.2
Changed lines of the file:
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@@
 <net name="RXD" class="0">
-<segment>
-<pinref part="SJ1" gate="1" pin="2"/>
-<wire x1="358.14" y1="53.34" x2="363.22" y2="53.34" width="0.1524" layer="91"/>
-<label x="363.22" y="53.34" size="1.27" layer="95" xref="yes"/>
-</segment>
 <segment>
 <label x="370.84" y="236.22" size="1.27" layer="95" xref="yes"/>
@@
 <label x="279.4" y="134.62" size="1.27" layer="95" rot="R180" xref="yes"/>
 </segment>
-</net>
-<net name="TXD" class="0">
 <segment>
 <pinref part="SJ2" gate="1" pin="2"/>
@@
 <label x="363.22" y="48.26" size="1.27" layer="95" xref="yes"/>
 </segment>
+</net>
+<net name="TXD" class="0">
 <segment>
 <wire x1="365.76" y1="233.68" x2="370.84" y2="233.68" width="0.1524" layer="91"/>
@@
 <label x="279.4" y="137.16" size="1.27" layer="95" rot="R180" xref="yes"/>
 </segment>
+<segment>
+<pinref part="SJ1" gate="1" pin="2"/>
+<wire x1="358.14" y1="53.34" x2="363.22" y2="53.34" width="0.1524" layer="91"/>
+<label x="363.22" y="53.34" size="1.27" layer="95" xref="yes"/>
+</segment>
 </net>

Commit message: Added interrupt signal,option between XIN and XOUT
Parts:
- removed LED1: green, SparkFun:LED0603
- removed R14: 1k, sven:RES-0402
- added SJ7: (no value), jumper:SJ2W
Connections:
- new net IRQ: IC2.11_NIRQ, IC4.PIO0_2/SSEL0/CT16B0_CAP0
- net GND: no longer R14.2
- net N$10: now also IC2.17_XIN, SJ7.3; no longer LED1.C, R14.1
- net N$17: now also IC2.16_XOUT, SJ7.1; no longer IC4.PIO0_2/SSEL0/CT16B0_CAP0, LED1.A
- net N$2: now also SJ7.2; no longer IC2.16_XOUT
Other:
- moved on the sheet: C24
Changed lines of the file:
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@@
 </variantdefs>
 <classes>
-<class number="0" name="default" width="0.1524" drill="0.3">
+<class number="0" name="default" width="0.15" drill="0.3">
 <clearance class="0" value="0.1524"/>
 </class>
@@
 <part name="P+5" library="SparkFun" deviceset="3.3V" device="" value="VCC"/>
 <part name="GND9" library="SparkFun" deviceset="GND" device=""/>
-<part name="LED1" library="SparkFun" deviceset="LED" device="0603" value="green">
-<attribute name="MF" value=""/>
-<attribute name="MPN" value=""/>
-<attribute name="OC_NEWARK" value="unknown"/>
-</part>
-<part name="GND17" library="SparkFun" deviceset="GND" device=""/>
 <part name="C27" library="sven" deviceset="CAP-0402" device="" value="4.7pF"/>
 <part name="C12" library="sven" deviceset="CAP-0805" device="" value="22uF"/>
@@
 <part name="C15" library="sven" deviceset="CAP-0402" device="" value="100pF"/>
 <part name="C1" library="sven" deviceset="CAP-0603" device="" value="2.2uF"/>
-<part name="R14" library="sven" deviceset="RES-0402" device="" value="1k"/>
 <part name="R5" library="sven" deviceset="RES-0402" device="" value="1k"/>
 <part name="C22" library="sven" deviceset="CAP-0402" device="" value="100pF"/>
@@
 <part name="GND39" library="SparkFun" deviceset="GND" device=""/>
 <part name="U$3" library="ava" deviceset="JTI_ANTENNA-1575AT43A40" device=""/>
+<part name="SJ7" library="jumper" deviceset="SJ2W" device=""/>
 </parts>
 <sheets>
@@
 <instance part="P+5" gate="G$1" x="441.96" y="165.1"/>
 <instance part="GND9" gate="1" x="441.96" y="127"/>
-<instance part="LED1" gate="G$1" x="251.46" y="203.2" rot="R180">
-<attribute name="OC_NEWARK" x="251.46" y="203.2" size="1.778" layer="96" display="off"/>
-<attribute name="MF" x="251.46" y="203.2" size="1.778" layer="96" display="off"/>
-<attribute name="MPN" x="251.46" y="203.2" size="1.778" layer="96" display="off"/>
-</instance>
-<instance part="GND17" gate="1" x="251.46" y="226.06" rot="R180"/>
 <instance part="C27" gate="G$1" x="99.06" y="111.76" rot="R90"/>
 <instance part="C12" gate="G$1" x="317.5" y="302.26"/>
@@
 <instance part="C15" gate="G$1" x="167.64" y="63.5" rot="R90"/>
 <instance part="C1" gate="G$1" x="116.84" y="276.86"/>
-<instance part="R14" gate="G$1" x="251.46" y="215.9" rot="R90"/>
 <instance part="R5" gate="G$1" x="363.22" y="58.42"/>
 <instance part="C22" gate="G$1" x="228.6" y="175.26" rot="R270"/>
-<instance part="C24" gate="G$1" x="208.28" y="170.18"/>
+<instance part="C24" gate="G$1" x="200.66" y="175.26" rot="R270"/>
 <instance part="C18" gate="G$1" x="210.82" y="246.38" rot="R270"/>
 <instance part="C19" gate="G$1" x="228.6" y="236.22" rot="R180"/>
@@
 <instance part="GND39" gate="1" x="177.8" y="198.12" rot="R180"/>
 <instance part="U$3" gate="G$1" x="284.48" y="93.98" rot="R90"/>
+<instance part="SJ7" gate="G$1" x="205.74" y="165.1" rot="R270"/>
 </instances>
 <busses>
@@
 <wire x1="441.96" y1="129.54" x2="441.96" y2="132.08" width="0.1524" layer="91"/>
 <pinref part="R9" gate="G$1" pin="1"/>
-</segment>
-<segment>
-<pinref part="GND17" gate="1" pin="GND"/>
-<wire x1="251.46" y1="220.98" x2="251.46" y2="223.52" width="0.1524" layer="91"/>
-<pinref part="R14" gate="G$1" pin="2"/>
 </segment>
 <segment>
@@
 <pinref part="VCXO" gate="G$1" pin="OUT"/>
 <wire x1="208.28" y1="182.88" x2="208.28" y2="175.26" width="0.1524" layer="91"/>
-<wire x1="208.28" y1="175.26" x2="208.28" y2="172.72" width="0.1524" layer="91"/>
+<wire x1="208.28" y1="175.26" x2="203.2" y2="175.26" width="0.1524" layer="91"/>
 <junction x="208.28" y="175.26"/>
 <wire x1="208.28" y1="175.26" x2="223.52" y2="175.26" width="0.1524" layer="91"/>
 <pinref part="C24" gate="G$1" pin="2"/>
 <pinref part="C22" gate="G$1" pin="1"/>
-</segment>
-</net>
-<net name="N$2" class="0">
-<segment>
-<pinref part="IC2" gate="G$1" pin="16_XOUT"/>
-<wire x1="208.28" y1="165.1" x2="208.28" y2="157.48" width="0.1524" layer="91"/>
-<pinref part="C24" gate="G$1" pin="1"/>
 </segment>
 </net>
@@
 </segment>
 </net>
-<net name="N$10" class="0">
-<segment>
-<pinref part="LED1" gate="G$1" pin="C"/>
-<wire x1="251.46" y1="208.28" x2="251.46" y2="210.82" width="0.1524" layer="91"/>
-<pinref part="R14" gate="G$1" pin="1"/>
-</segment>
-</net>
 <net name="ADC_VSOL" class="0">
 <segment>
@@
 </segment>
 </net>
-<net name="N$17" class="0">
-<segment>
-<pinref part="LED1" gate="G$1" pin="A"/>
-<pinref part="IC4" gate="G$1" pin="PIO0_2/SSEL0/CT16B0_CAP0"/>
-<wire x1="251.46" y1="200.66" x2="251.46" y2="198.12" width="0.1524" layer="91"/>
-<wire x1="251.46" y1="198.12" x2="279.4" y2="198.12" width="0.1524" layer="91"/>
-</segment>
-</net>
 <net name="I2C_PULL_VCC" class="0">
 <segment>
@@
 </segment>
 </net>
+<net name="IRQ" class="0">
+<segment>
+<pinref part="IC2" gate="G$1" pin="11_NIRQ"/>
+<wire x1="238.76" y1="96.52" x2="243.84" y2="96.52" width="0.1524" layer="91"/>
+<label x="243.84" y="96.52" size="1.27" layer="95" xref="yes"/>
+</segment>
+<segment>
+<pinref part="IC4" gate="G$1" pin="PIO0_2/SSEL0/CT16B0_CAP0"/>
+<wire x1="279.4" y1="198.12" x2="274.32" y2="198.12" width="0.1524" layer="91"/>
+<label x="274.32" y="198.12" size="1.27" layer="95" rot="R180" xref="yes"/>
+</segment>
+</net>
+<net name="N$2" class="0">
+<segment>
+<pinref part="C24" gate="G$1" pin="1"/>
+<wire x1="195.58" y1="175.26" x2="193.04" y2="175.26" width="0.1524" layer="91"/>
+<pinref part="SJ7" gate="G$1" pin="2"/>
+<wire x1="193.04" y1="175.26" x2="193.04" y2="170.18" width="0.1524" layer="91"/>
+<wire x1="193.04" y1="170.18" x2="205.74" y2="170.18" width="0.1524" layer="91"/>
+</segment>
+</net>
+<net name="N$10" class="0">
+<segment>
+<pinref part="SJ7" gate="G$1" pin="3"/>
+<pinref part="IC2" gate="G$1" pin="17_XIN"/>
+<wire x1="200.66" y1="165.1" x2="200.66" y2="157.48" width="0.1524" layer="91"/>
+</segment>
+</net>
+<net name="N$17" class="0">
+<segment>
+<pinref part="SJ7" gate="G$1" pin="1"/>
+<wire x1="210.82" y1="165.1" x2="210.82" y2="160.02" width="0.1524" layer="91"/>
+<wire x1="210.82" y1="160.02" x2="208.28" y2="160.02" width="0.1524" layer="91"/>
+<pinref part="IC2" gate="G$1" pin="16_XOUT"/>
+<wire x1="208.28" y1="160.02" x2="208.28" y2="157.48" width="0.1524" layer="91"/>
+</segment>
+</net>
