File: PecanPico6.sch (EAGLE design)
At the start: 79 parts, among them IC1 TPS79718DCKT, IC2 SI4463/4, IC3 UBLOX_MAX-6, IC4 LPC1114FHN33/333, IC5 SPV1040, IC6 AS213-92LF, IC7 BMP180, Q2 AP2301

Commit message: Initial commit of new PecanPico6b degin
Parts:
- removed JP5: (no value), pinhead:PINHD-2X6
- removed LED2: red, SparkFun:LED0603
- removed LED3: blue, SparkFun:LED0603
- removed R13, R5: 1k, sven:RES-0402
- removed R17: 22k, sven:RES-0402
- removed R18: 10k, sven:RES-0402
- removed SJ1, SJ2, SJ3, SJ4, SJ5: (no value), jumper:SJ
- removed SJ7: (no value), jumper:SJ2W
- removed TP1, TP2: TPTP07R, testpad:TPTP07R
- added C8: 100nF, sven:CAP-0402
- added JP1, JP6, JP7: (no value), pinhead:PINHD-2X4
Connections:
- removed net ADC_VSOL: IC4.R/PIO1_0/AD1/CT32B1_CAP0, R17.1, R18.2
- removed net LDO_EN: IC1.PG, IC4.R/PIO1_2/AD3/CT32B1_MAT1
- removed net N$15: IC3.3_RXD1, SJ1.1
- removed net N$2: C24.1, SJ7.2
- removed net N$20: IC3.2_TXD1, SJ2.1
- removed net N$25: IC3.16_SDA2, SJ3.2
- removed net N$26: IC3.17_SCL2, SJ4.2
- removed net N$4: C22.2, IC4.XTALIN
- removed net N$6: LED2.C, R5.2
- removed net N$8: IC3.4_TIMEPULSE, R5.1
- removed net N$9: LED3.C, R13.2
- new net TIMEPULSE: IC3.4_TIMEPULSE, IC4.PIO1_11/AD7/CT32B1_CAP1
- net GND: now also C8.1, JP1.6, JP1.7; no longer JP5.10, JP5.11, JP5.12, JP5.3, R13.1, R18.1, TP2.TP
- net I2C_PULL_VCC: now also IC4.PIO0_3; no longer IC4.PIO1_9/CT16B1_MAT0/MOSI1
- net ISP_ENTRY: no longer TP1.TP
- net N$10: now also C24.1; no longer SJ7.3
- net N$13: now also C22.2; no longer C22.1
- net N$17: now also C22.1; no longer SJ7.1
- net N$5: now also C8.2; no longer SJ5.1
- net OUT1: no longer JP5.8
- net OUT2: now also IC4.R/PIO1_2/AD3/CT32B1_MAT1; no longer IC4.PIO1_11/AD7/CT32B1_CAP1, JP5.6
- net OUT3: no longer JP5.4
- net OUT4: no longer JP5.2
- net RESET: now also JP1.1; no longer JP5.5
- net RXD: no longer SJ2.2
- net SCL: now also IC3.17_SCL2, JP1.4; no longer SJ4.1
- net SDA: now also IC3.16_SDA2, JP1.2; no longer SJ3.1
- net SWCLK: now also JP1.5; no longer JP5.9
- net SWDIO: now also JP1.3; no longer JP5.7
- net TXD: no longer SJ1.2
- net TX_EN: no longer LED3.A
- net VCC15: now also IC1.PG, JP1.8; no longer JP5.1, LED2.A, SJ5.2
- net VCXO_EN: now also IC4.PIO1_9/CT16B1_MAT0/MOSI1; no longer IC4.PIO0_3
- net VSOLAR: now also IC4.R/PIO1_0/AD1/CT32B1_CAP0; no longer R17.2
Other:
- note removed: "Pull low to"
- note removed: "activate ISP"
- moved on the sheet: C18, C19, C21, C22, C24, C25, R10, R11, R12, R16, SJ8, VCXO

Commit message: Moved microcontroller
Parts:
- removed C25, C8: 100nF, sven:CAP-0402
- removed R7: 10k, sven:RES-0402
- removed UART: PINHEAD_PINHD-1X10S, 1_27x3:PINHEAD_PINHD-1X10S
- removed VCXO: OSCILLATORSMD6, SparkFun-FreqCtrl_TK:OSCILLATORSMD6
- added U$2: VCXO, sven:VCXO
Connections:
- removed net ISP_ENTRY: IC4.PIO0_1/CLKOUT/CT32B0_MAT2
- removed net OUT1: IC4.PIO1_4/AD5/CT32B1_MAT3/WAKEUP, JP2.3
- removed net OUT2: IC4.R/PIO1_2/AD3/CT32B1_MAT1, JP2.4
- removed net OUT3: IC4.PIO3_2/CT16B0_MAT2/SCK1, JP2.5
- removed net OUT4: IC4.PIO1_5/RTS/CT32B0_CAP0, JP2.6
- net GND: now also U$2.GND; no longer C25.1, C8.1, UART.3, VCXO.GND
- net GPIO0: now also IC4.PIO3_5/CT16B1_CAP1/TXD; no longer IC4.PIO3_4/CT16B0_CAP1/RXD
- net GPIO1: now also IC4.PIO3_4/CT16B0_CAP1/RXD; no longer IC4.PIO3_5/CT16B1_CAP1/TXD
- net GPS_OFF: now also IC4.PIO2_0/DTR/SSEL1; no longer IC4.PIO1_8/CT16B1_CAP0
- net GPS_RESET: now also IC4.PIO1_8/CT16B1_CAP0; no longer IC4.PIO2_0/DTR/SSEL1, R7.1
- net I2C_PULL_VCC: now also IC4.R/PIO1_2/AD3/CT32B1_MAT1; no longer IC4.PIO0_3
- net IRQ: now also IC4.PIO1_10/AD6/CT16B1_MAT1/MISO1; no longer IC4.PIO0_2/SSEL0/CT16B0_CAP0
- net N$13: now also U$2.OUT; no longer VCXO.OUT
- net N$14: now also U$2.VCC; no longer VCXO.VCC
- net N$21: now also U$2.AFC; no longer VCXO.VC
- net N$5: no longer C25.2, C8.2
- net RADIO_SDN: no longer IC4.PIO1_10/AD6/CT16B1_MAT1/MISO1
- net RXD: no longer UART.2
- net TXD: no longer UART.1
- net VCC15: no longer R7.2, SJ8.1
- net VCXO_EN: now also SJ8.1; no longer IC4.PIO1_9/CT16B1_MAT0/MOSI1, VCXO.EN
Other:
- moved on the sheet: C18, C19, C21, R10, R11, R12, R16, SJ8

Commit message: Sorted parts
Parts:
- removed IC3: UBLOX_MAX-6, ava:UBLOX_MAX-6
- removed U$3: JTI_ANTENNA-1575AT43A40, ava:JTI_ANTENNA-1575AT43A40
- added U$4: UBLOX_CAM, ava:UBLOX_CAM
Connections:
- removed net N$3: IC3.11_RF_IN, U$3.FEED
- new net N$2: U$4.16_ANT, U$4.17_RF_IN
- net GND: now also U$4.GND; no longer IC3.10_GND, IC3.12_GND, IC3.1_GND, JP1.6
- net GPIO0: now also IC4.PIO1_7/TXD/CT32B0_MAT1; no longer IC4.PIO3_5/CT16B1_CAP1/TXD
- net GPIO1: now also IC4.PIO1_6/RXD/CT32B0_MAT0; no longer IC4.PIO3_4/CT16B0_CAP1/RXD
- net GPS_OFF: now also IC4.PIO1_4/AD5/CT32B1_MAT3/WAKEUP; no longer IC4.PIO2_0/DTR/SSEL1
- net GPS_RESET: now also IC4.PIO0_2/SSEL0/CT16B0_CAP0, U$4.23/RESET_N; no longer IC3.9_V_RESET, IC4.PIO1_8/CT16B1_CAP0
- net I2C_PULL_VCC: now also IC4.PIO0_3; no longer IC4.R/PIO1_2/AD3/CT32B1_MAT1
- net IRQ: now also IC4.PIO1_5/RTS/CT32B0_CAP0; no longer IC4.PIO1_10/AD6/CT16B1_MAT1/MISO1
- net N$5: now also U$4.9/VCC; no longer IC3.8_VCC
- net RXD: now also IC4.PIO3_4/CT16B0_CAP1/RXD; no longer IC4.PIO1_6/RXD/CT32B0_MAT0
- net SCL: now also U$4.6/SCL; no longer IC3.17_SCL2, JP1.4
- net SDA: now also U$4.3/SDA; no longer IC3.16_SDA2, JP1.2
- net SS: now also IC4.PIO2_0/DTR/SSEL1; no longer IC4.PIO0_7/CTS
- net TIMEPULSE: now also IC4.PIO0_7/CTS, U$4.29/TIMEPULSE; no longer IC3.4_TIMEPULSE, IC4.PIO1_11/AD7/CT32B1_CAP1
- net TXD: now also IC4.PIO3_5/CT16B1_CAP1/TXD; no longer IC4.PIO1_7/TXD/CT32B0_MAT1
- net VCC15: now also U$4.1/VCC_IO, U$4.8/V_BCKUP; no longer IC3.6_V_BCKP, IC3.7_VCC_IO, JP1.8
- net VCC1V8: now also IC4.PIO1_10/AD6/CT16B1_MAT1/MISO1
- net VSOLAR: now also IC4.R/PIO1_2/AD3/CT32B1_MAT1; no longer IC4.R/PIO1_0/AD1/CT32B1_CAP0

Commit message: Done some more sorting
Parts:
- removed C17: 2.2uF, sven:CAP-0603
- removed JP2: (no value), PecanPico5a:PINHD-1X10
- removed U$4: UBLOX_CAM, ava:UBLOX_CAM
- added C8: 2.2uF, sven:CAP-0402
- added U$3: UBLOX_CAM, Ava:UBLOX_CAM
- C1: device sven:CAP-0603 -> sven:CAP-0402
Connections:
- net GND: now also C1.2, C8.1, U$3.GND; no longer C1.1, C17.2, JP2.10, U$4.GND
- net GPIO0: no longer IC4.PIO1_7/TXD/CT32B0_MAT1
- net GPIO1: now also IC4.PIO1_7/TXD/CT32B0_MAT1; no longer IC4.PIO1_6/RXD/CT32B0_MAT0
- net GPS_RESET: now also U$3.23/RESET_N; no longer U$4.23/RESET_N
- net IRQ: now also IC4.PIO1_6/RXD/CT32B0_MAT0; no longer IC4.PIO1_5/RTS/CT32B0_CAP0
- net N$2: now also U$3.16_ANT, U$3.17_RF_IN; no longer U$4.16_ANT, U$4.17_RF_IN
- net N$5: now also U$3.9/VCC; no longer U$4.9/VCC
- net RESET: no longer JP2.8
- net RXD: now also JP1.4
- net SCL: now also U$3.6/SCL; no longer U$4.6/SCL
- net SDA: now also U$3.3/SDA; no longer U$4.3/SDA
- net SS: now also IC4.PIO1_5/RTS/CT32B0_CAP0; no longer IC4.PIO2_0/DTR/SSEL1
- net SWCLK: no longer JP2.1
- net SWDIO: no longer JP2.2
- net TIMEPULSE: now also U$3.29/TIMEPULSE; no longer U$4.29/TIMEPULSE
- net TXD: now also JP1.2
- net VCC15: now also C1.1, U$3.1/VCC_IO, U$3.8/V_BCKUP; no longer C17.1, JP2.9, U$4.1/VCC_IO, U$4.8/V_BCKUP
- net VCC1V8: now also C8.2; no longer C1.2, IC4.R/PIO1_1/AD2/CT32B1_MAT0
- net VCXO_CTRL: now also IC4.R/PIO1_1/AD2/CT32B1_MAT0; no longer IC4.R/PIO0_11/AD0/CT32B0_MAT3
Other:
- moved on the sheet: C1

Commit message: Moved stuff around the PCB
Connections:
- net GND: now also JP1.6
- net GPS_OFF: now also IC4.PIO0_3; no longer IC4.PIO1_4/AD5/CT32B1_MAT3/WAKEUP
- net I2C_PULL_VCC: now also IC4.PIO1_9/CT16B1_MAT0/MOSI1; no longer IC4.PIO0_3
- net RXD: no longer JP1.4
- net SCL: now also JP1.4
- net SDA: now also JP1.2
- net TXD: no longer JP1.2
- net VCC15: now also JP1.8
- net VSOLAR: now also IC4.PIO1_11/AD7/CT32B1_CAP1; no longer IC4.R/PIO1_2/AD3/CT32B1_MAT1
Changed lines of the file:
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@@
 <part name="C1" library="sven" deviceset="CAP-0402" device="" value="2.2uF"/>
 <part name="U$3" library="Ava" deviceset="UBLOX_CAM" device=""/>
+<part name="P+6" library="SparkFun" deviceset="3.3V" device="" value="VCC"/>
+<part name="GND6" library="SparkFun" deviceset="GND" device=""/>
 </parts>
 <sheets>
@@
 <instance part="C1" gate="G$1" x="167.64" y="43.18" rot="R90"/>
 <instance part="U$3" gate="G$1" x="325.12" y="63.5"/>
+<instance part="P+6" gate="G$1" x="469.9" y="142.24" rot="R270"/>
+<instance part="GND6" gate="1" x="480.06" y="127"/>
 </instances>
 <busses>
@@
 <wire x1="477.52" y1="111.76" x2="477.52" y2="96.52" width="0.1524" layer="91"/>
 <pinref part="GND13" gate="1" pin="GND"/>
+</segment>
+<segment>
+<pinref part="JP1" gate="A" pin="6"/>
+<wire x1="462.28" y1="144.78" x2="480.06" y2="144.78" width="0.1524" layer="91"/>
+<wire x1="480.06" y1="144.78" x2="480.06" y2="129.54" width="0.1524" layer="91"/>
+<pinref part="GND6" gate="1" pin="GND"/>
 </segment>
 </net>
@@
 <pinref part="P+8" gate="G$1" pin="3.3V"/>
 </segment>
+<segment>
+<pinref part="JP1" gate="A" pin="8"/>
+<wire x1="462.28" y1="142.24" x2="469.9" y2="142.24" width="0.1524" layer="91"/>
+<pinref part="P+6" gate="G$1" pin="3.3V"/>
+</segment>
 </net>
 <net name="SDA" class="0">
@@
 <wire x1="462.28" y1="116.84" x2="469.9" y2="116.84" width="0.1524" layer="91"/>
 </segment>
+<segment>
+<pinref part="JP1" gate="A" pin="2"/>
+<wire x1="462.28" y1="149.86" x2="469.9" y2="149.86" width="0.1524" layer="91"/>
+<label x="469.9" y="149.86" size="1.27" layer="95" xref="yes"/>
+</segment>
 </net>
 <net name="SS" class="0">
@@
 <segment>
 <wire x1="462.28" y1="114.3" x2="469.9" y2="114.3" width="0.1524" layer="91"/>
+</segment>
+<segment>
+<pinref part="JP1" gate="A" pin="4"/>
+<wire x1="462.28" y1="147.32" x2="469.9" y2="147.32" width="0.1524" layer="91"/>
+<label x="469.9" y="147.32" size="1.27" layer="95" xref="yes"/>
 </segment>
 </net>
@@
 </segment>
 <segment>
-<pinref part="IC4" gate="G$1" pin="R/PIO1_2/AD3/CT32B1_MAT1"/>
-<wire x1="292.1" y1="223.52" x2="287.02" y2="223.52" width="0.1524" layer="91"/>
-<label x="287.02" y="223.52" size="1.27" layer="95" rot="R180" xref="yes"/>
+<label x="287.02" y="210.82" size="1.27" layer="95" rot="R180" xref="yes"/>
+<pinref part="IC4" gate="G$1" pin="PIO1_11/AD7/CT32B1_CAP1"/>
+<wire x1="287.02" y1="210.82" x2="292.1" y2="210.82" width="0.1524" layer="91"/>
 </segment>
 </net>
@@
 </segment>
 <segment>
-<pinref part="IC4" gate="G$1" pin="PIO1_4/AD5/CT32B1_MAT3/WAKEUP"/>
-<wire x1="292.1" y1="185.42" x2="287.02" y2="185.42" width="0.1524" layer="91"/>
-<label x="287.02" y="185.42" size="1.27" layer="95" rot="R180" xref="yes"/>
+<pinref part="IC4" gate="G$1" pin="PIO0_3"/>
+<wire x1="292.1" y1="190.5" x2="287.02" y2="190.5" width="0.1524" layer="91"/>
+<label x="287.02" y="190.5" size="1.27" layer="95" rot="R180" xref="yes"/>
 </segment>
 </net>
@@
 </segment>
 <segment>
-<pinref part="IC4" gate="G$1" pin="PIO0_3"/>
-<wire x1="292.1" y1="190.5" x2="287.02" y2="190.5" width="0.1524" layer="91"/>
-<label x="287.02" y="190.5" size="1.27" layer="95" rot="R180" xref="yes"/>
+<pinref part="IC4" gate="G$1" pin="PIO1_9/CT16B1_MAT0/MOSI1"/>
+<wire x1="378.46" y1="208.28" x2="383.54" y2="208.28" width="0.1524" layer="91"/>
+<label x="383.54" y="208.28" size="1.27" layer="95" xref="yes"/>
 </segment>
 </net>
@@
 <label x="383.54" y="228.6" size="1.27" layer="95" xref="yes"/>
 </segment>
-<segment>
-<pinref part="JP1" gate="A" pin="2"/>
-<wire x1="462.28" y1="149.86" x2="469.9" y2="149.86" width="0.1524" layer="91"/>
-<label x="469.9" y="149.86" size="1.27" layer="95" xref="yes"/>
-</segment>
 </net>
 <net name="RXD" class="0">
@@
 <label x="383.54" y="226.06" size="1.27" layer="95" xref="yes"/>
 </segment>
-<segment>
-<pinref part="JP1" gate="A" pin="4"/>
-<wire x1="462.28" y1="147.32" x2="469.9" y2="147.32" width="0.1524" layer="91"/>
-<label x="469.9" y="147.32" size="1.27" layer="95" xref="yes"/>
-</segment>
-</net>
+</net>
