File: PecanPico6.brd (EAGLE design)
At the start: 50 x 29.8 mm, 79 parts, among them IC1 TPS79718DCKT, IC2 SI4463/4, IC3 UBLOX_MAX-6, IC4 LPC1114FHN33/333, IC5 SPV1040, IC6 AS213-92LF, IC7 BMP180, Q2 AP2301

Commit message: Created version 6b Removed RX part Removed UART pinheader below GPS module Enlarged Solar pad Fixed VCC_IO pin connection at GPS Enlarged Board for holes
Parts:
- removed C27, C4: 4.7pF, sven:0402
- removed C3, L8, R19: (no value), sven:0402
- removed IC6: AS213-92LF, sven:SC-70
- removed L6, L7: 56nH, sven:0402
- removed U$3: JTI_ANTENNA-1575AT43A40, ava:JTI_ANTENNA-1575AT43A40
- removed UART: PINHEAD_PINHD-1X10S, 1_27x3:PINHEAD_1X10S
- added JP1: GPSANTENNA, sven:PAD2_1.8X0.9
- moved JP3 0.50 mm to (10.4, 9.75)
Connections:
- removed net GND: C1.P$1, C11.P$1, C12.P$1, C13.P$1, C14.P$1, C15.P$2, C16.P$2, C17.P$2, C18.P$1, C2.P$1, C20.P$1, C21.P$1, C25.P$1, C27.P$2, C5.P$1, C6.P$1, C7.P$1, C9.P$1, IC1.2, IC2.18, IC2.21, IC2.22, IC2.23, IC2.24, IC2.25, IC2.5, IC3.10_GND, IC3.12_GND, IC3.1_GND, IC4.33, IC5.2, IC6.2, IC7.7, JP2.10, JP5.10, JP5.11, JP5.12, JP5.3, R12.P$1, R13.P$1, R18.P$1, R19.P$1, R2.P$1, R9.P$1, TP2.TP, U$1.GND1, U$1.GND2, U$1.GND3, UART.P$3, VCXO.3, VCXO.3INNER
- removed net N$16: C3.P$1, L8.P$1, R19.P$2
- removed net N$24: C4.P$1, IC2.2, L6.P$2
- removed net N$33: C27.P$1, IC2.3, L6.P$1, L7.P$1
- removed net N$37: C4.P$2, IC6.3, L7.P$2
- removed net N$5: C25.P$2, IC3.8_VCC, Q2.3, SJ5.1
- new net N$100: C1.P$1, C11.P$1, C12.P$1, C13.P$1, C14.P$1, C15.P$2, C16.P$2, C17.P$2, C18.P$1, C2.P$1, C20.P$1, C21.P$1, C25.P$1, C5.P$1, C6.P$1, C7.P$1, C9.P$1, IC1.2, IC2.18, IC2.21, IC2.22, IC2.23, IC2.24, IC2.25, IC2.5, IC3.10_GND, IC3.12_GND, IC3.1_GND, IC4.33, IC5.2, IC7.7, JP2.10, JP5.10, JP5.11, JP5.12, JP5.3, R12.P$1, R13.P$1, R18.P$1, R2.P$1, R9.P$1, TP2.TP, U$1.GND1, U$1.GND2, U$1.GND3, VCXO.3, VCXO.3INNER
- net N$1: now also L3.P$1; no longer IC6.5
- net N$11: now also C25.P$2, IC3.7_VCC_IO, IC3.8_VCC, Q2.3, SJ5.1; no longer IC6.1, L3.P$1
- net N$27: no longer C3.P$2, L8.P$2
- net N$3: now also JP1.1; no longer U$3.FEED
- net RXD: no longer UART.P$2
- net RX_EN: no longer IC6.4
- net TXD: no longer UART.P$1
- net TX_EN: no longer IC6.6
- net VCC15: no longer IC3.7_VCC_IO
Routing:
- net GND: track 37.6 -> 0.00 mm, vias 54 -> 0
- net N$100: track 0.00 -> 25.3 mm, vias 0 -> 61
- net N$5: track 16.9 -> 0.00 mm, vias 2 -> 1
- net N$11: track 1.08 -> 16.8 mm, vias 0 -> 2
- net RX_EN: track 5.77 -> 0.00 mm, vias 2 -> 0
- net TX_EN: track 6.98 -> 1.45 mm, vias 2 -> 0
- net RXD: track 14.0 -> 9.47 mm, vias 2 -> 1
- net N$33: track 3.38 -> 0.00 mm
- net N$1: track 2.15 -> 5.07 mm
- net N$24: track 2.20 -> 0.00 mm
- net N$27: track 2.92 -> 0.86 mm
- net TXD: track 10.9 -> 8.87 mm, vias 2 -> 1
- net N$37: track 1.92 -> 0.00 mm
- net N$16: track 1.86 -> 0.00 mm, vias 0 -> 1
- net VCC15: track 122.6 -> 121.5 mm
- added copper zone on layer 1, net N$100
- added copper zone on layer 16, net N$100
- removed copper zone on layer 1, net GND
- removed copper zone on layer 16, net GND
Other:
- board size 50 x 29.8 mm -> 52.1 x 22.7 mm
- board text added: "Version 02. November 2015"
- board text removed: "Version 03. April 2015"

Commit message: Moved solar pads
Parts:
- added JP6: M01SOLAR, sven:PAD2_1.8X0.9
- moved JP3 10.0 mm to (0.40, 10.4), turned to 90 degrees
Routing:
- net VSOLAR: track 22.0 -> 34.8 mm, vias 2 -> 4
Changed lines of the file:
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@@
 <layer number="23" name="tOrigins" color="15" fill="1" visible="yes" active="yes"/>
 <layer number="24" name="bOrigins" color="15" fill="1" visible="yes" active="yes"/>
-<layer number="25" name="tNames" color="7" fill="1" visible="yes" active="yes"/>
-<layer number="26" name="bNames" color="7" fill="1" visible="yes" active="yes"/>
+<layer number="25" name="tNames" color="7" fill="1" visible="no" active="yes"/>
+<layer number="26" name="bNames" color="7" fill="1" visible="no" active="yes"/>
 <layer number="27" name="tValues" color="7" fill="1" visible="no" active="yes"/>
 <layer number="28" name="bValues" color="7" fill="1" visible="no" active="yes"/>
@@
 <attribute name="VALUE" x="49.8999" y="17.6" size="0.02" layer="28" rot="MR0"/>
 </element>
-<element name="JP3" library="sven" package="PAD2_1.8X0.9" value="M01SOLAR" x="10.4" y="9.75">
-<attribute name="OC_NEWARK" value="unknown" x="10.4" y="9.75" size="1.778" layer="27" display="off"/>
-<attribute name="MF" value="" x="10.4" y="9.75" size="1.778" layer="27" display="off"/>
-<attribute name="MPN" value="" x="10.4" y="9.75" size="1.778" layer="27" display="off"/>
+<element name="JP3" library="sven" package="PAD2_1.8X0.9" value="M01SOLAR" x="0.4" y="10.4" rot="R90">
+<attribute name="OC_NEWARK" value="unknown" x="0.4" y="10.4" size="1.778" layer="27" rot="R90" display="off"/>
+<attribute name="MF" value="" x="0.4" y="10.4" size="1.778" layer="27" rot="R90" display="off"/>
+<attribute name="MPN" value="" x="0.4" y="10.4" size="1.778" layer="27" rot="R90" display="off"/>
 </element>
 <element name="JP4" library="sven" package="PAD3.5X7.0" value="M01BATTERY" x="47.5" y="15.2" rot="MR90">
@@
 <attribute name="MF" value="" x="49.75" y="22" size="1.778" layer="27" display="off"/>
 <attribute name="OC_NEWARK" value="unknown" x="49.75" y="22" size="1.778" layer="27" display="off"/>
+</element>
+<element name="JP6" library="sven" package="PAD2_1.8X0.9" value="M01SOLAR" x="0.4" y="19.1" rot="R90">
+<attribute name="MPN" value="" x="0.4" y="19.1" size="1.778" layer="27" rot="R90" display="off"/>
+<attribute name="MF" value="" x="0.4" y="19.1" size="1.778" layer="27" rot="R90" display="off"/>
+<attribute name="OC_NEWARK" value="unknown" x="0.4" y="19.1" size="1.778" layer="27" rot="R90" display="off"/>
 </element>
 </elements>
@@
 <wire x1="11.85" y1="17.75" x2="11.2" y2="17.1" width="0.3" layer="1"/>
 <wire x1="11.2" y1="17.1" x2="11.85" y2="16.45" width="0.3" layer="1"/>
-<via x="7.5" y="11.5" extent="1-16" drill="0.3"/>
 <via x="5" y="16.5" extent="1-16" drill="0.3"/>
 <via x="15.7" y="14.1" extent="1-16" drill="0.3"/>
@@
 <via x="7.8" y="13.9" extent="1-16" drill="0.3"/>
 <via x="5.4" y="14.3" extent="1-16" drill="0.3"/>
-<via x="5.6" y="12.2" extent="1-16" drill="0.3"/>
-<via x="6.4" y="11.9" extent="1-16" drill="0.3"/>
+<via x="5.3" y="12.4" extent="1-16" drill="0.3"/>
+<via x="6.3" y="12.2" extent="1-16" drill="0.3"/>
 <via x="6.7" y="14.2" extent="1-16" drill="0.3"/>
+<via x="11.4" y="11.4" extent="1-16" drill="0.3"/>
 </signal>
 <signal name="SCK">
@@
 <wire x1="22.65" y1="11.275" x2="22.325" y2="11.275" width="0.2" layer="1"/>
 <contactref element="JP3" pad="1"/>
-<wire x1="10.4" y1="9.75" x2="12.53" y2="9.75" width="0.6" layer="1"/>
 <wire x1="12.53" y1="9.75" x2="12.53" y2="10.6" width="0.6" layer="1"/>
 <wire x1="17.475" y1="11.275" x2="17.8" y2="11.6" width="0.2" layer="1"/>
@@
 <wire x1="18.5" y1="11" x2="17.9" y2="11.6" width="0.2" layer="1"/>
 <wire x1="17.9" y1="11.6" x2="17.8" y2="11.6" width="0.2" layer="1"/>
+<wire x1="12.4022375" y1="9.3292375" x2="12.4022375" y2="10.6" width="0.5" layer="1"/>
+<wire x1="12.4022375" y1="10.6" x2="10.2" y2="10.6" width="0.5" layer="1"/>
+<via x="10.2" y="10.6" extent="1-16" drill="0.3"/>
+<wire x1="10.2" y1="10.6" x2="7.7" y2="10.6" width="0.5" layer="16"/>
+<wire x1="7.7" y1="10.6" x2="7.1" y2="11.2" width="0.5" layer="16"/>
+<wire x1="7.1" y1="11.2" x2="6" y2="11.2" width="0.5" layer="16"/>
+<wire x1="6" y1="11.2" x2="3.9" y2="9.1" width="0.5" layer="16"/>
+<wire x1="3.9" y1="9.1" x2="1.7" y2="9.1" width="0.5" layer="16"/>
+<wire x1="1.7" y1="9.1" x2="0.4" y2="10.4" width="0.5" layer="16"/>
+<via x="0.4" y="10.4" extent="1-16" drill="0.3"/>
 </signal>
 <signal name="N$36">
@@
 <wire x1="43.2" y1="13.8" x2="40.2" y2="13.8" width="0.3" layer="1"/>
 </signal>
-<signal name="N$5">
-<via x="0.3" y="9.7" extent="1-16" drill="0.8"/>
-</signal>
 <signal name="N$16">
-<via x="0.3" y="12.2" extent="1-16" drill="0.8"/>
+<via x="0.3" y="13" extent="1-16" drill="0.8"/>
 </signal>
 <signal name="N$18">
@@
 </signal>
 <signal name="N$19">
-<via x="0.3" y="17.3" extent="1-16" drill="0.8"/>
-</signal>
-<signal name="N$22">
-<via x="0.3" y="19.8" extent="1-16" drill="0.8"/>
+<via x="0.3" y="16.5" extent="1-16" drill="0.8"/>
 </signal>
 </signals>
